File: CTS-SAT-1-Burnwire-PCB-KiCad/CTS-SAT-1-Burnwire-PCB-KiCad.kicad_pcb (KiCad board)
At the start: 2 copper layers, 50.8 x 22.9 mm, 20 parts, among them J1 feather long, J2 feather short, U1 ADP2303ARDZ

Commit message: Update CTS-SAT-1-Burnwire-PCB-KiCad.kicad_pcb
Parts:
- moved R4 1.30 mm to (60.0, 41.0)
Changed lines of the file:
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@@
 	(footprint "Resistor_SMD:R_0201_0603Metric"
 		(layer "F.Cu")
-		(at 61.32 40.86 180)
+		(at 60.035 41.03 180)
 		(descr "Resistor SMD 0201 (0603 Metric), square (rectangular) end terminal, IPC_7351 nominal, (Body size source: https://www.vishay.com/docs/20052/crcw0201e3.pdf), generated with kicad-footprint-generator")
 		(tags "resistor")
